File: PCB/Air_pump_controler/Air_pump_controler.kicad_pcb (KiCad board)
At the start: 2 copper layers, 24 x 24 mm, 21 parts, among them J1 Conn_01x03_Pin, J2 USB IN, J3 Cable mount, J4 Motor_conn, Q1 AP30N03DF, U1 CH32V003F4U6

Commit message: Update
PCB shematic and layout done rev.:0.1
Parts:
- removed C2: 4.7uF, Capacitor_SMD:C_0603_1608Metric
- removed J3: Cable mount, Connector_PinHeader_2.54mm:PinHeader_1x02_P2.54mm_Vertical
- added C5: 4.7uF, Capacitor_SMD:C_0402_1005Metric, F.Cu at (158.5, 81.5)
- added C6: TBD, Capacitor_SMD:C_0603_1608Metric, F.Cu at (160.4, 92.4)
- added D1: 1N4148W, Diode_SMD:D_SOD-123, F.Cu at (161.9, 89.6)
- added D2: PWR, LED_SMD:LED_0603_1608Metric, F.Cu at (158.8, 79.8)
- added R8: TBD, Resistor_SMD:R_0603_1608Metric, F.Cu at (160.4, 95.5)
- added R9: 100, Resistor_SMD:R_0603_1608Metric, F.Cu at (155.7, 79.8)
- moved R3 36.6 mm to (151.1, 96.2), turned to -90 degrees
- moved R4 36.4 mm to (151.1, 93.0), turned to -90 degrees
- moved C8 30.3 mm to (157.2, 87.5)
- moved C3 28.1 mm to (151.1, 89.9), turned to -90 degrees
- moved C1 25.7 mm to (153.2, 95.5), turned to 90 degrees
- moved C9 25.7 mm to (162.9, 82.1)
- moved R5 24.6 mm to (162.9, 97.6), turned to 180 degrees
- moved TH1 23.4 mm to (165.3, 92.4), turned to -90 degrees
- moved R6 22.6 mm to (165.3, 95.5), turned to 90 degrees
- moved C4 20.9 mm to (153.2, 90.7), turned to -90 degrees
- moved C10 20.5 mm to (160.3, 85.7), turned to -90 degrees
- moved L1 16.9 mm to (156.9, 91.2), turned to 90 degrees
- moved R7 16.6 mm to (162.9, 96.0), turned to 180 degrees
- moved J2 14.5 mm to (156.9, 96.2), turned to 0 degrees
- moved U1 5.10 mm to (157.2, 84.2), turned to 180 degrees
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Connections:
- C3 pad 1: Net-(J4-Pin_2) -> Net-(D1-K)
- C4 pad 1: Net-(J4-Pin_2) -> Net-(D1-K)
- J4 pad 1: (no net) -> Net-(D1-A)
- J4 pad 2: (no net) -> Net-(D1-K)
- L1 pad 2: Net-(J4-Pin_2) -> Net-(D1-K)
- Q1 pad 3: Net-(J4-Pin_1) -> Net-(D1-A)
- U1 pad 11: unconnected-(U1-PC4-Pad11) -> /LED
- U1 pad 15: unconnected-(U1-PD1-Pad15) -> /SWIO
- U1 pad 16: unconnected-(U1-PD2-Pad16) -> /LS_SW
- U1 pad 2: unconnected-(U1-PA1-Pad2) -> /AN_TEMP
- U1 pad 20: unconnected-(U1-PD6-Pad20) -> /AN_V_IN
- U1 pad 3: unconnected-(U1-PA2-Pad3) -> /AN_POT
Routing:
- net +5V: track 0.00 -> 55.9 mm, vias 0 -> 4
- net /LS_SW: track 0.00 -> 15.7 mm, vias 0 -> 2
- net /AN_V_IN: track 0.00 -> 15.5 mm, vias 0 -> 2
- net /AN_TEMP: track 0.00 -> 14.9 mm, vias 0 -> 2
- net GND: track 0.00 -> 10.3 mm, vias 0 -> 36
- net Net-(D1-K): track 0.00 -> 9.40 mm
- net /AN_POT: track 0.00 -> 7.17 mm
- net /SWIO: track 0.00 -> 6.43 mm
- net /LED: track 0.00 -> 4.39 mm
- net Net-(Q1-G): track 0.00 -> 3.15 mm
- net Net-(C6-Pad2): track 0.00 -> 1.50 mm
- net Net-(D2-A): track 0.00 -> 1.49 mm
- net Net-(D1-A): track 0.00 -> 1.40 mm
- added copper zone on F.Cu, net Net-(D1-A)
- added copper zone on F.Cu, net Net-(D1-K)
Other:
- board text added: "+5V"
- board text added: "-ADJ-"
- board text added: "5V"
- board text added: "Air pump control Designed by: Tinta T. October 2025"
- board text added: "GND"
- board text added: "JLCJLCJLCJLC"
- board text added: "SWIO"

Commit message: Finished PCB
Parts:
- added RX: U_RX, TestPoint:TestPoint_Pad_D1.0mm, F.Cu at (154.6, 87.3)
- added TX: U_TX, TestPoint:TestPoint_Pad_D1.0mm, F.Cu at (152.3, 87.3)
- moved C8 5.81 mm to (154.2, 82.5), turned to 90 degrees
- moved J1 1.59 mm to (149.3, 84.5), turned to 60 degrees
- moved C10 0.82 mm to (160.6, 84.8)
- moved C9 0.25 mm to (163.0, 81.8)
- moved RV1 0.25 mm to (163.9, 84.5)
Connections:
- U1 pad 10: unconnected-(U1-PC3-Pad10) -> /LED
- U1 pad 11: /LED -> /AN_V_IN
- U1 pad 19: unconnected-(U1-PD5-Pad19) -> Net-(U1-PD5)
- U1 pad 20: /AN_V_IN -> Net-(U1-PD6)
Routing:
- net Net-(D1-K): track 9.40 -> 0.39 mm
- net Net-(U1-PD5): track 0.00 -> 7.08 mm
- net Net-(U1-PD6): track 0.00 -> 5.14 mm
- net GND: track 10.3 -> 7.08 mm
- net /AN_TEMP: track 14.9 -> 17.3 mm
- net +5V: track 55.9 -> 56.7 mm
- net /AN_POT: track 7.17 -> 7.99 mm
- net /LED: track 4.39 -> 3.60 mm
- net /AN_V_IN: track 15.5 -> 16.2 mm
- net /SWIO: track 6.43 -> 7.00 mm
